File: hardware/pcb/battery-powered-smart-vision-module/_restore_backup_2026-07-08T16-23-27-717/battery-powered-smart-vision-module.kicad_pcb (KiCad board)
At the start: 2 copper layers, 72.5 x 40.5 mm, 15 parts, among them J1 Conn_01x02, J3 I2C Header, J4 GPIO Header, SW2 SW_SPST

Commit message: Complete PCB design updates and hardware integration
Updated KiCad schematic, PCB layout, custom XIAO ESP32S3 Sense footprint, project files, manufacturing outputs, and hardware documentation. Continued development of the battery-powered smart vision module.
Changed lines of the file:
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@@
 		(filling no)
 		(pcbplotparams
-			(layerselection 0x00000000_00000000_55555555_57555573)
+			(layerselection 0x00000000_00000000_55555555_5755f5ff)
 			(plot_on_all_layers_selection 0x00000000_00000000_00000000_00000000)
 			(disableapertmacros no)
@@
 			(outputformat 1)
 			(mirror no)
-			(drillshape 0)
+			(drillshape 1)
 			(scaleselection 1)
-			(outputdirectory "../../Gerbers/")
+			(outputdirectory "")
 		)
 	)
@@
 		(tags "resistor")
 		(property "Reference" "R4"
-			(at -2.0875 -4 0)
-			(layer "F.SilkS")
-			(effects
+			(at -2.0875 -6.5 0)
+			(layer "F.SilkS")
+			(effects
