File: hardware/pcb/battery-powered-smart-vision-module_backup_before_xiao_fix/battery-powered-smart-vision-module_backup_before_xiao_fix.kicad_pcb (KiCad board)
At the start: 2 copper layers, 72.5 x 40.5 mm, 15 parts, among them J1 Conn_01x02, J3 I2C Header, J4 GPIO Header, SW2 SW_SPST

Commit message: Complete Revision A PCB design and manufacturing files
Complete Revision A PCB design and manufacturing files
Parts:
- added J2: I2C Header, Connector_PinHeader_2.54mm:PinHeader_1x04_P2.54mm_Vertical, F.Cu at (64.0, 78.0)
- TP1: value BAT -> 3V3
- TP2: value 3V3 -> 5V; footprint TestPoint:TestPoint_Loop_D3.80mm_Drill2.8mm -> TestPoint:TestPoint_2Pads_Pitch2.54mm_Drill0.8mm
- TP3: footprint TestPoint:TestPoint_Loop_D3.80mm_Drill2.8mm -> TestPoint:TestPoint_2Pads_Pitch2.54mm_Drill0.8mm
Connections:
- J4 pad 1: Net-(J4-Pin_1) -> +5V
- J4 pad 2: Net-(J4-Pin_2) -> Net-(J4-GND)
- J4 pad 3: Net-(J4-Pin_3) -> Net-(J4-3V3)
- J4 pad 4: Net-(J4-Pin_4) -> Net-(J2-Pin_2)
- J4 pad 5: Net-(J4-Pin_5) -> Net-(J4-D1)
- J4 pad 6: Net-(J4-Pin_6) -> Net-(J4-D2)
- J4 pad 7: Net-(J4-Pin_7) -> Net-(J4-D3)
- J4 pad 8: Net-(J4-Pin_8) -> Net-(J4-D6_(TX))
- R4 pad 1: Net-(D2-K) -> Net-(J2-Pin_2)
- R4 pad 2: Net-(J4-Pin_8) -> Net-(D2-K)
- TP1 pad 1: Net-(J1-Pin_1) -> Net-(J2-Pin_2)
- TP2 pad 1: +3.3V -> +5V
- U1 pad 10: unconnected-(U1-A3-Pad10) -> Net-(J4-D1)
- U1 pad 11: Net-(J4-Pin_1) -> Net-(J2-Pin_3)
- U1 pad 12: Net-(J4-Pin_2) -> Net-(J4-D2)
- U1 pad 13: Net-(J4-Pin_3) -> Net-(J4-D6_(TX))
- U1 pad 14: Net-(J4-Pin_4) -> Net-(J4-D3)
- U1 pad 2: +3.3V -> +5V
- U1 pad 4: Net-(J3-Pin_1) -> Net-(J4-GND)
- U1 pad 5: Net-(J3-Pin_3) -> unconnected-(U1-D2_(GPIO3)-Pad5)
- U1 pad 6: Net-(J3-Pin_4) -> Net-(J4-3V3)
- U1 pad 8: unconnected-(U1-A1-Pad8) -> Net-(J2-Pin_2)
- U1 pad 9: unconnected-(U1-A2-Pad9) -> Net-(J2-Pin_4)
Routing:
- net (no net): track 0.00 -> 79.5 mm
- net Net-(J4-Pin_3): track 28.2 -> 0.00 mm
- net Net-(J4-Pin_2): track 19.0 -> 0.00 mm
- net Net-(J4-Pin_1): track 17.1 -> 0.00 mm
- net Net-(J4-Pin_4): track 15.2 -> 0.00 mm
- net Net-(J4-Pin_8): track 5.76 -> 0.00 mm
- net Net-(D2-K): track 7.21 -> 13.0 mm
