File: hardware/pcb/Battery-Powered-Smart-Vision-Module_Final/Battery-Powered-Smart-Vision-Module_Final.kicad_sch (KiCad schematic)
At the start: 12 parts, among them J2 GPIO Header, J3 I2C Header, J4 Conn_01x07, J5 Conn_01x07

Commit message: Release Rev A
 Finalized PCB layout
- Updated schematic and title blocks
- Generated manufacturing Gerbers
- CNC milled PCB
- Hand assembled prototype
- Verified power operation
- ESP32-S3 detected over USB
Other:
- company: (none) -> Hovering Horizons LLC
- title: (none) -> Battery Powered Smart Vision Module
Changed lines of the file:
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@@
 	(generator_version "10.0")
 	(paper "A4")
+	(title_block
+		(title "Battery Powered Smart Vision Module")
+		(date "Released July 2026")
+		(rev "Revision A")
+		(company "Hovering Horizons LLC")
+		(comment 1 "Project: Sure Sight Security")
+		(comment 2 "Board: Seeed Studio XIAO ESP32-S3 Sense")
+		(comment 3 "Designed by Trinity Matthew Ison")
+	)
 	(junction
 		(at 147.32 60.96)
